File: Discharger_ConstantCurrent/Schematic/Discharger_ConstantCurrent/Discharger_ConstantCurrent.kicad_sch (KiCad schematic)
At the start: 23 parts, among them J1 Input 1, J2 Input 2, Q1 IPD80R1K0CEATMA1, U1 LR8K4-G

Commit message: File cleanup
Parts:
- R2: value 1kΩ 1W -> 100Ω 1W
Changed lines of the file:
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@@
       (effects (font (size 1.27 1.27)))
     )
-    (property "Value" "1kΩ 1W" (at 74.295 48.26 90)
+    (property "Value" "100Ω 1W" (at 74.295 48.26 90)
       (effects (font (size 1.27 1.27)))
     )
